File: hardware/stk3700-cc1101/GG-CC1101_v1.2.brd (EAGLE design)
At the start: 40.6 x 28 mm, 18 parts, among them U1 CC1101, X1 BU-SMA-V

Commit message: updated schema
Parts:
- C10, C9: value 22P -> 13pF
- turned JP1 to 180 degrees
- renumbered JP2 to JP1, U$2 to Q1
Connections:
- net 3V3: now also JP1.2; no longer JP1.1
- net CSN: now also JP1.10; no longer JP1.11
- net GDO0: now also JP1.5; no longer JP1.16
- net GDO2: now also JP1.7; no longer JP1.14
- net GND: now also JP1.1; no longer JP1.2, JP1.20
- net SCLK: now also JP1.8; no longer JP1.13
- net SI: now also JP1.4; no longer JP1.17
- net SO: now also JP1.6; no longer JP1.15
Routing:
- net 3V3: track 56.0 -> 30.3 mm
Other:
- board text added: "CC1101_GG_v1.2"
