File: hardware/stk3700-cc1101/GG-CC1101_v1.2.sch (EAGLE design)
At the start: 18 parts, among them U1 CC1101, X1 BU-SMA-V

Commit message: updated schema
Parts:
- removed JP2: (no value), pinhead:PINHD-2X10
- added JP1: (no value), pinhead:PINHD-2X10
- C10, C9: value 22P -> 13pF
- renumbered U$2 to Q1
Connections:
- net 3V3: now also JP1.2; no longer JP2.1
- net CSN: now also JP1.10; no longer JP2.11
- net GDO0: now also JP1.5; no longer JP2.16
- net GDO2: now also JP1.7; no longer JP2.14
- net GND: now also JP1.1; no longer JP2.2, JP2.20
- net SCLK: now also JP1.8; no longer JP2.13
- net SI: now also JP1.4; no longer JP2.17
- net SO: now also JP1.6; no longer JP2.15
Changed lines of the file:
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@@
 <setting verticaltext="up"/>
 </settings>
-<grid distance="1" unitdist="mil" unit="mil" style="lines" multiple="1" display="yes" altdistance="0.01" altunitdist="inch" altunit="inch"/>
+<grid distance="0.1" unitdist="inch" unit="inch" style="lines" multiple="1" display="no" altdistance="0.01" altunitdist="inch" altunit="inch"/>
 <layers>
 <layer number="1" name="Top" color="4" fill="1" visible="no" active="no"/>
@@
 <part name="GND10" library="SparkFun" deviceset="GND" device=""/>
 <part name="GND11" library="SparkFun" deviceset="GND" device=""/>
-<part name="JP2" library="pinhead" deviceset="PINHD-2X10" device=""/>
-<part name="GND14" library="SparkFun" deviceset="GND" device=""/>
-<part name="GND15" library="SparkFun" deviceset="GND" device=""/>
-<part name="C9" library="SparkFun" deviceset="CAP" device="0805" value="22P"/>
-<part name="C10" library="SparkFun" deviceset="CAP" device="0805" value="22P"/>
+<part name="C9" library="SparkFun" deviceset="CAP" device="0805" value="13pF"/>
+<part name="C10" library="SparkFun" deviceset="CAP" device="0805" value="13pF"/>
 <part name="GND12" library="SparkFun" deviceset="GND" device=""/>
 <part name="GND13" library="SparkFun" deviceset="GND" device=""/>
-<part name="U$2" library="Dragan-Personal" deviceset="XTAL-26MHZ" device=""/>
+<part name="Q1" library="Dragan-Personal" deviceset="XTAL-26MHZ" device=""/>
 <part name="GND16" library="SparkFun" deviceset="GND" device=""/>
 <part name="GND17" library="SparkFun" deviceset="GND" device=""/>
+<part name="JP1" library="pinhead" deviceset="PINHD-2X10" device=""/>
+<part name="GND19" library="SparkFun" deviceset="GND" device=""/>
 </parts>
 <sheets>
@@
 <instance part="GND10" gate="1" x="152.4508" y="40.8686"/>
 <instance part="GND11" gate="1" x="243.8908" y="40.8686"/>
-<instance part="JP2" gate="A" x="30.5308" y="43.4086"/>
-<instance part="GND14" gate="1" x="43.2308" y="58.6486" rot="R180"/>
-<instance part="GND15" gate="1" x="43.2308" y="25.6286"/>
 <instance part="C9" gate="G$1" x="91.4908" y="56.1086" smashed="yes">
 <attribute name="NAME" x="91.7448" y="59.0296" size="1.778" layer="95"/>
@@
 <instance part="GND12" gate="1" x="91.4908" y="45.9486"/>
 <instance part="GND13" gate="1" x="116.8908" y="45.9486"/>
-<instance part="U$2" gate="G$1" x="101.6508" y="63.7286"/>
+<instance part="Q1" gate="G$1" x="101.6508" y="63.7286"/>
 <instance part="GND16" gate="1" x="101.6508" y="53.5686"/>
 <instance part="GND17" gate="1" x="106.7308" y="53.5686"/>
+<instance part="JP1" gate="A" x="30.48" y="40.64" rot="R180"/>
+<instance part="GND19" gate="1" x="40.64" y="22.86"/>
 </instances>
 <busses>
@@
 </segment>
 <segment>
-<pinref part="JP2" gate="A" pin="13"/>
-<wire x1="27.9908" y1="38.3286" x2="20.3708" y2="38.3286" width="0.1524" layer="91"/>
-<label x="20.3708" y="38.3286" size="1.778" layer="95" rot="R180"/>
+<pinref part="JP1" gate="A" pin="8"/>
+<wire x1="25.4" y1="38.1" x2="17.78" y2="38.1" width="0.1524" layer="91"/>
+<label x="17.78" y="38.1" size="1.778" layer="95" rot="R180"/>
 </segment>
 </net>
@@
 </segment>
 <segment>
-<pinref part="JP2" gate="A" pin="15"/>
-<wire x1="27.9908" y1="35.7886" x2="20.3708" y2="35.7886" width="0.1524" layer="91"/>
-<label x="20.3708" y="35.7886" size="1.778" layer="95" rot="R180"/>
+<pinref part="JP1" gate="A" pin="6"/>
+<wire x1="25.4" y1="35.56" x2="17.78" y2="35.56" width="0.1524" layer="91"/>
+<label x="17.78" y="35.56" size="1.778" layer="95" rot="R180"/>
 </segment>
 </net>
@@
 </segment>
 <segment>
-<pinref part="JP2" gate="A" pin="14"/>
-<wire x1="35.6108" y1="38.3286" x2="43.2308" y2="38.3286" width="0.1524" layer="91"/>
-<label x="43.2308" y="38.3286" size="1.778" layer="95"/>
+<pinref part="JP1" gate="A" pin="7"/>
+<wire x1="33.02" y1="38.1" x2="40.64" y2="38.1" width="0.1524" layer="91"/>
+<label x="40.64" y="38.1" size="1.778" layer="95"/>
 </segment>
 </net>
@@
 </segment>
 <segment>
-<pinref part="JP2" gate="A" pin="2"/>
-<pinref part="GND14" gate="1" pin="GND"/>
-<wire x1="35.6108" y1="53.5686" x2="43.2308" y2="53.5686" width="0.1524" layer="91"/>
-<wire x1="43.2308" y1="53.5686" x2="43.2308" y2="56.1086" width="0.1524" layer="91"/>
-</segment>
-<segment>
-<pinref part="JP2" gate="A" pin="20"/>
-<pinref part="GND15" gate="1" pin="GND"/>
-<wire x1="35.6108" y1="30.7086" x2="43.2308" y2="30.7086" width="0.1524" layer="91"/>
-<wire x1="43.2308" y1="30.7086" x2="43.2308" y2="28.1686" width="0.1524" layer="91"/>
-</segment>
-<segment>
 <pinref part="GND12" gate="1" pin="GND"/>
 <pinref part="C9" gate="G$1" pin="2"/>
@@
 </segment>
 <segment>
-<pinref part="U$2" gate="G$1" pin="P$2"/>
+<pinref part="Q1" gate="G$1" pin="P$2"/>
 <pinref part="GND16" gate="1" pin="GND"/>
 <wire x1="101.6508" y1="56.1086" x2="101.6508" y2="58.6486" width="0.1524" layer="91"/>
 </segment>
 <segment>
-<pinref part="U$2" gate="G$1" pin="P$4"/>
+<pinref part="Q1" gate="G$1" pin="P$4"/>
 <pinref part="GND17" gate="1" pin="GND"/>
 <wire x1="106.7308" y1="56.1086" x2="106.7308" y2="58.6486" width="0.1524" layer="91"/>
+</segment>
+<segment>
+<wire x1="40.64" y1="30.48" x2="40.64" y2="25.4" width="0.1524" layer="91"/>
+<pinref part="GND19" gate="1" pin="GND"/>
+<pinref part="JP1" gate="A" pin="1"/>
+<wire x1="40.64" y1="30.48" x2="33.02" y2="30.48" width="0.1524" layer="91"/>
 </segment>
 </net>
@@
 </segment>
 <segment>
-<pinref part="JP2" gate="A" pin="17"/>
-<wire x1="27.9908" y1="33.2486" x2="20.3708" y2="33.2486" width="0.1524" layer="91"/>
-<label x="20.3708" y="33.2486" size="1.778" layer="95" rot="R180"/>
+<pinref part="JP1" gate="A" pin="4"/>
+<wire x1="25.4" y1="33.02" x2="17.78" y2="33.02" width="0.1524" layer="91"/>
+<label x="17.78" y="33.02" size="1.778" layer="95" rot="R180"/>
 </segment>
 </net>
@@
 <wire x1="91.4908" y1="61.1886" x2="91.4908" y2="63.7286" width="0.1524" layer="91"/>
 <label x="91.4908" y="66.2686" size="1.778" layer="95"/>
-<pinref part="U$2" gate="G$1" pin="P$1"/>
+<pinref part="Q1" gate="G$1" pin="P$1"/>
 <wire x1="91.4908" y1="63.7286" x2="91.4908" y2="66.2686" width="0.1524" layer="91"/>
 <wire x1="96.5708" y1="63.7286" x2="91.4908" y2="63.7286" width="0.1524" layer="91"/>
@@
 <wire x1="116.8908" y1="61.1886" x2="116.8908" y2="63.7286" width="0.1524" layer="91"/>
 <label x="116.8908" y="66.2686" size="1.778" layer="95"/>
-<pinref part="U$2" gate="G$1" pin="P$3"/>
+<pinref part="Q1" gate="G$1" pin="P$3"/>
 <wire x1="116.8908" y1="63.7286" x2="116.8908" y2="66.2686" width="0.1524" layer="91"/>
 <wire x1="111.8108" y1="63.7286" x2="116.8908" y2="63.7286" width="0.1524" layer="91"/>
@@
 </segment>
 <segment>
-<pinref part="JP2" gate="A" pin="11"/>
-<wire x1="27.9908" y1="40.8686" x2="20.3708" y2="40.8686" width="0.1524" layer="91"/>
-<label x="20.3708" y="40.8686" size="1.778" layer="95" rot="R180"/>
+<pinref part="JP1" gate="A" pin="10"/>
+<wire x1="25.4" y1="40.64" x2="17.78" y2="40.64" width="0.1524" layer="91"/>
+<label x="17.78" y="40.64" size="1.778" layer="95" rot="R180"/>
 </segment>
 </net>
@@
 </segment>
 <segment>
-<pinref part="JP2" gate="A" pin="16"/>
-<wire x1="35.6108" y1="35.7886" x2="43.2308" y2="35.7886" width="0.1524" layer="91"/>
-<label x="43.2308" y="35.7886" size="1.778" layer="95"/>
+<pinref part="JP1" gate="A" pin="5"/>
+<wire x1="33.02" y1="35.56" x2="40.64" y2="35.56" width="0.1524" layer="91"/>
+<label x="40.64" y="35.56" size="1.778" layer="95"/>
 </segment>
 </net>
@@
 </segment>
 <segment>
-<pinref part="JP2" gate="A" pin="1"/>
-<wire x1="27.9908" y1="53.5686" x2="20.3708" y2="53.5686" width="0.1524" layer="91"/>
-<label x="20.3708" y="53.5686" size="1.778" layer="95" rot="R180"/>
-</segment>
-</net>
+<pinref part="JP1" gate="A" pin="2"/>
+<wire x1="25.4" y1="30.48" x2="17.78" y2="30.48" width="0.1524" layer="91"/>
+<label x="17.78" y="30.48" size="1.778" layer="95" rot="R180"/>
+</segment>
+</net>
